File: schematic/bhm/_autosave-bhm.kicad_sch (KiCad schematic)
At the start: 12 parts, among them J1 Conn_01x04, U1 LM358, U2 ATtiny45-20P, U3 LM78L05_TO92

Commit message: testing out generating some preliminary pcb layouts
Parts:
- added R6, R8: 30k, Resistor_THT:R_Axial_DIN0207_L6.3mm_D2.5mm_P7.62mm_Horizontal, symbol Device:R
- added R7, R9: 4.7M, Resistor_THT:R_Axial_DIN0207_L6.3mm_D2.5mm_P7.62mm_Horizontal, symbol Device:R
- added SENS: .01, Resistor_SMD:R_0201_0603Metric_Pad0.64x0.40mm_HandSolder, symbol Device:R
- added unit 2 of U1
Connections:
- net +8.4V: now also R8.2, SENS.1
- net GND: now also R9.1
- net at U2.3 (XTAL2/PB4): now also R7.1, U1.7
- new net: R8.1, R9.2, U1.5 (+)
- new net: R6.1, R7.2, U1.6 (-)
- new net: R6.2, SENS.2
