File: schematic/bhm/bhm.kicad_pcb (KiCad board)
At the start: 2 copper layers, 11 parts, among them J1 Conn_01x04, U1 LM358, U2 ATtiny45-20P, U3 LM78L05_TO92

Commit message: finalized v1 schematic and PCB layout
Parts:
- added C3: 100nf, Capacitor_THT:C_Radial_D4.0mm_H7.0mm_P1.50mm, F.Cu at (235.8, 132.9)
- added G***: LOGO, LOGO, B.Cu at (215.8, 135.5)
- added NegBatt1: Conn_01x01, 1_Custom_Pads:bhm_large_power_pad, F.Cu at (197.0, 132.0)
- added NegDevice1: Conn_01x01, 1_Custom_Pads:bhm_large_power_pad, F.Cu at (256.0, 132.0)
- added PosBatt1: Conn_01x01, 1_Custom_Pads:bhm_large_power_pad, F.Cu at (197.0, 122.0)
- added PosDevice1: Conn_01x01, 1_Custom_Pads:bhm_large_power_pad, F.Cu at (256.0, 122.0)
- added R6: 22k, Resistor_THT:R_Axial_DIN0207_L6.3mm_D2.5mm_P7.62mm_Horizontal, F.Cu at (231.1, 132.0)
- added R7: 220k, Resistor_THT:R_Axial_DIN0207_L6.3mm_D2.5mm_P7.62mm_Horizontal, F.Cu at (231.1, 128.0)
- added SENS1: .01, Resistor_SMD:R_2816_7142Metric_Pad3.20x4.45mm_HandSolder, F.Cu at (216.6, 137.0)
- C1: footprint Capacitor_THT:C_Radial_D4.0mm_H7.0mm_P1.50mm -> Capacitor_THT:C_Disc_D3.0mm_W1.6mm_P2.50mm
- C2: footprint Capacitor_THT:C_Disc_D5.0mm_W2.5mm_P5.00mm -> Capacitor_THT:C_Disc_D3.0mm_W1.6mm_P2.50mm
- moved R1 109.6 mm to (235.5, 121.2), turned to -90 degrees
- moved U2 101.7 mm to (238.7, 124.2)
- moved U1 96.7 mm to (212.9, 122.4)
- moved J1 93.4 mm to (249.5, 123.0)
- moved U3 88.4 mm to (229.5, 121.0), turned to 180 degrees
- moved R2 84.3 mm to (209.5, 125.0), turned to 180 degrees
- moved R4 83.9 mm to (209.5, 132.0), turned to 180 degrees
- moved R3 82.0 mm to (209.5, 122.0), turned to 180 degrees
- moved C1 78.2 mm to (224.0, 124.0)
- moved C2 75.5 mm to (232.5, 124.0), turned to 180 degrees
- moved R5 74.4 mm to (201.9, 129.0)
Connections:
- C2 pad 1: Net-(J1-Pin_3) -> /5v
- J1 pad 1: Net-(J1-Pin_1) -> GND
- J1 pad 2: Net-(J1-Pin_2) -> /5v
- J1 pad 4: GND -> Net-(J1-Pin_4)
- R1 pad 1: Net-(J1-Pin_3) -> /5v
- R3 pad 1: Net-(J1-Pin_3) -> /5v
- U1 pad 5: (no net) -> Net-(NegDevice1-Pin_1)
- U1 pad 6: (no net) -> Net-(U1B--)
- U1 pad 7: (no net) -> Net-(U2-XTAL2/PB4)
- U2 pad 3: unconnected-(U2-XTAL2/PB4-Pad3) -> Net-(U2-XTAL2/PB4)
- U2 pad 5: Net-(J1-Pin_1) -> Net-(J1-Pin_4)
- U2 pad 7: Net-(J1-Pin_2) -> Net-(J1-Pin_3)
- U2 pad 8: Net-(J1-Pin_3) -> /5v
- U3 pad 1: Net-(J1-Pin_3) -> /5v
Routing:
- net GND: track 0.00 -> 155.5 mm, vias 0 -> 11
- net +8.4V: track 0.00 -> 151.6 mm, vias 0 -> 10
- net Net-(NegDevice1-Pin_1): track 0.00 -> 84.0 mm, vias 0 -> 11
- net /5v: track 0.00 -> 70.3 mm
- net Net-(U2-XTAL1/PB3): track 0.00 -> 40.1 mm
- net Net-(U2-XTAL2/PB4): track 0.00 -> 21.0 mm
- net Net-(U1A--): track 0.00 -> 16.2 mm
- net Net-(U1B--): track 0.00 -> 12.5 mm
- net Net-(U1A-+): track 0.00 -> 7.02 mm
- net Net-(U2-~{RESET}/PB5): track 0.00 -> 5.94 mm
- net Net-(J1-Pin_3): track 0.00 -> 3.74 mm
- net Net-(J1-Pin_4): track 0.00 -> 3.68 mm
Other:
- board outline added: 67 x 24.5 mm
- board text added: "+"
- board text added: "-"
- board text added: "Battery Monitor Rev. v0.1"
- board text added: "Design by: M. Hautman"
- board text added: "batt"
- board text added: "device"
