File: schematic/bhm/bhm.kicad_sch (KiCad schematic)
At the start: 19 parts, among them J1 Conn_01x04, U1 LM358, U2 ATtiny45-20P, U3 LM78L05_TO92

Commit message: finalized v1 schematic and PCB layout
Parts:
- C1: footprint Capacitor_THT:C_Radial_D4.0mm_H7.0mm_P1.50mm -> Capacitor_THT:C_Disc_D3.0mm_W1.6mm_P2.50mm
- C2: footprint Capacitor_THT:C_Disc_D5.0mm_W2.5mm_P5.00mm -> Capacitor_THT:C_Disc_D3.0mm_W1.6mm_P2.50mm
- C3: footprint (none) -> Capacitor_THT:C_Radial_D4.0mm_H7.0mm_P1.50mm
- J1: value Conn_01x04 -> SSD1306
- NegBatt1: renamed from NegBatt; footprint (none) -> 1_Custom_Pads:bhm_large_power_pad
- NegDevice1: renamed from NegDevice; footprint (none) -> 1_Custom_Pads:bhm_large_power_pad
- PosBatt1: renamed from PosBatt; footprint (none) -> 1_Custom_Pads:bhm_large_power_pad
- PosDevice1: renamed from PosDevice; footprint (none) -> 1_Custom_Pads:bhm_large_power_pad
- SENS1: renamed from SENS; footprint Resistor_SMD:R_0201_0603Metric_Pad0.64x0.40mm_HandSolder -> Resistor_SMD:R_2816_7142Metric_Pad3.20x4.45mm_HandSolder
- U1: footprint (none) -> Package_DIP:DIP-8_W7.62mm
Connections:
- net GND: now also J1.1 (Pin_1); no longer J1.4 (Pin_4)
- net 5v: now reaches C2.1, C3.1, R1.1, R3.1, U2.8 (VCC), U3.1 (VO)
- net 5v: now also J1.2 (Pin_2); no longer J1.3 (Pin_3)
- net at U2.5 (AREF/PB0): now also J1.4 (Pin_4); no longer J1.1 (Pin_1)
- net at U2.7 (PB2): now also J1.3 (Pin_3); no longer J1.2 (Pin_2)
Other:
- moved on the sheet: J1
Changed lines of the file:
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@@
-	(wire
-		(pts
-			(xy 138.43 88.9) (xy 138.43 119.38)
-		)
-		(stroke
-			(width 0)
-			(type default)
-		)
-	)
-	(wire
-		(pts
-			(xy 135.89 91.44) (xy 135.89 121.92)
-		)
-		(stroke
-			(width 0)
-			(type default)
-		)
-	)
-	(wire
-		(pts
-			(xy 130.81 119.38) (xy 130.81 121.92)
-		)
-		(stroke
-			(width 0)
-			(type default)
-		)
-	)
 	(wire
 		(pts
@@
 	(wire
 		(pts
+			(xy 130.81 116.84) (xy 130.81 127)
+		)
+		(stroke
+			(width 0)
+			(type default)
+		)
+	)
+	(wire
+		(pts
 			(xy 128.27 101.6) (xy 140.97 101.6)
 		)
@@
 	(wire
 		(pts
+			(xy 135.89 91.44) (xy 135.89 114.3)
+		)
+		(stroke
+			(width 0)
+			(type default)
+		)
+	)
+	(wire
+		(pts
+			(xy 138.43 121.92) (xy 133.35 121.92)
+		)
+		(stroke
+			(width 0)
+			(type default)
+		)
+	)
+	(wire
+		(pts
 			(xy 160.02 110.49) (xy 163.83 110.49)
 		)
@@
 	(wire
 		(pts
-			(xy 128.27 121.92) (xy 128.27 119.38)
-		)
-		(stroke
-			(width 0)
-			(type default)
-		)
-	)
-	(wire
-		(pts
 			(xy 88.9 119.38) (xy 113.03 119.38)
 		)
@@
 	(wire
 		(pts
-			(xy 138.43 119.38) (xy 130.81 119.38)
-		)
-		(stroke
-			(width 0)
-			(type default)
-		)
-	)
-	(wire
-		(pts
 			(xy 154.94 80.01) (xy 154.94 81.28)
 		)
@@
 	(wire
 		(pts
-			(xy 133.35 96.52) (xy 133.35 121.92)
-		)
-		(stroke
-			(width 0)
-			(type default)
-		)
-	)
-	(wire
-		(pts
 			(xy 163.83 119.38) (xy 166.37 119.38)
 		)
@@
 	(wire
 		(pts
+			(xy 133.35 116.84) (xy 130.81 116.84)
+		)
+		(stroke
+			(width 0)
+			(type default)
+		)
+	)
+	(wire
+		(pts
 			(xy 163.83 124.46) (xy 163.83 127)
 		)
@@
 	(wire
 		(pts
+			(xy 128.27 114.3) (xy 128.27 127)
+		)
+		(stroke
+			(width 0)
+			(type default)
+		)
+	)
+	(wire
+		(pts
 			(xy 147.32 121.92) (xy 147.32 110.49)
 		)
@@
 	(wire
 		(pts
+			(xy 135.89 114.3) (xy 128.27 114.3)
+		)
+		(stroke
+			(width 0)
+			(type default)
+		)
+	)
+	(wire
+		(pts
 			(xy 128.27 99.06) (xy 158.75 99.06)
 		)
@@
 	(wire
 		(pts
-			(xy 128.27 119.38) (xy 113.03 119.38)
+			(xy 113.03 119.38) (xy 135.89 119.38)
+		)
+		(stroke
+			(width 0)
+			(type default)
+		)
+	)
+	(wire
+		(pts
+			(xy 133.35 121.92) (xy 133.35 127)
 		)
 		(stroke
@@
 	(wire
 		(pts
+			(xy 135.89 119.38) (xy 135.89 127)
+		)
+		(stroke
+			(width 0)
+			(type default)
+		)
+	)
+	(wire
+		(pts
+			(xy 133.35 96.52) (xy 133.35 116.84)
+		)
+		(stroke
+			(width 0)
+			(type default)
+		)
+	)
+	(wire
+		(pts
 			(xy 158.75 99.06) (xy 163.83 99.06)
 		)
@@
 	(wire
 		(pts
+			(xy 138.43 88.9) (xy 138.43 121.92)
+		)
+		(stroke
+			(width 0)
+			(type default)
+		)
+	)
+	(wire
+		(pts
 			(xy 173.99 106.68) (xy 173.99 114.3)
 		)
@@
 			(width 0)
 			(type default)
+		)
+	)
+	(label "5v"
+		(at 113.03 78.74 0)
+		(fields_autoplaced yes)
+		(effects
+			(font
+				(size 1.27 1.27)
+			)
+			(justify left bottom)
+		)
+		(property "5v" ""
+			(at 113.03 80.01 0)
+			(effects
+				(font
+					(size 1.27 1.27)
+					(italic yes)
+				)
+				(justify left)
+			)
+		)
+	)
+	(label "5v"
+		(at 113.03 78.74 0)
+		(fields_autoplaced yes)
+		(effects
+			(font
+				(size 1.27 1.27)
+			)
+			(justify left bottom)
+		)
+		(property "+5V" ""
+			(at 113.03 80.01 0)
+			(effects
+				(font
+					(size 1.27 1.27)
+					(italic yes)
+				)
+				(justify left)
+			)
 		)
 	)
@@
 			)
 		)
-		(property "Footprint" ""
+		(property "Footprint" "Package_DIP:DIP-8_W7.62mm"
 			(at 154.94 121.92 0)
 			(effects
@@
 		(dnp no)
 		(fields_autoplaced yes)
-		(property "Reference" "NegDevice"
+		(property "Reference" "NegDevice1"
 			(at 187.96 123.1899 0)
 			(effects
@@
 			)
 		)
-		(property "Footprint" ""
+		(property "Footprint" "1_Custom_Pads:bhm_large_power_pad"
 			(at 185.42 124.46 0)
 			(effects
@@
 			(project "bhm"
 				(path "/6523cac7-11e3-4c79-8b92-51f4f81b827e"
-					(reference "NegDevice")
+					(reference "NegDevice1")
 					(unit 1)
 				)
@@
 		(dnp no)
 		(fields_autoplaced yes)
-		(property "Reference" "PosDevice"
+		(property "Reference" "PosDevice1"
 			(at 187.96 71.1199 0)
 			(effects
@@
 			)
 		)
-		(property "Footprint" ""
+		(property "Footprint" "1_Custom_Pads:bhm_large_power_pad"
 			(at 185.42 72.39 0)
 			(effects
@@
 			(project "bhm"
 				(path "/6523cac7-11e3-4c79-8b92-51f4f81b827e"
-					(reference "PosDevice")
+					(reference "PosDevice1")
 					(unit 1)
 				)
@@
 		(dnp no)
 		(fields_autoplaced yes)
-		(property "Reference" "NegBatt"
+		(property "Reference" "NegBatt1"
 			(at 187.96 134.6199 0)
 			(effects
@@
 			)
 		)
-		(property "Footprint" ""
+		(property "Footprint" "1_Custom_Pads:bhm_large_power_pad"
 			(at 185.42 135.89 0)
 			(effects
@@
 			(project "bhm"
 				(path "/6523cac7-11e3-4c79-8b92-51f4f81b827e"
-					(reference "NegBatt")
+					(reference "NegBatt1")
 					(unit 1)
 				)
@@
 			)
 		)
-		(property "Footprint" "Capacitor_THT:C_Radial_D4.0mm_H7.0mm_P1.50mm"
+		(property "Footprint" "Capacitor_THT:C_Disc_D3.0mm_W1.6mm_P2.50mm"
 			(at 164.7952 81.28 0)
 			(effects
@@
 			)
 		)
-		(property "Footprint" "Capacitor_THT:C_Disc_D5.0mm_W2.5mm_P5.00mm"
+		(property "Footprint" "Capacitor_THT:C_Disc_D3.0mm_W1.6mm_P2.50mm"
 			(at 145.0848 81.28 0)
 			(effects
@@
 					(size 1.27 1.27)
 				)
+				(hide yes)
 			)
 		)
@@
 			)
 		)
-		(property "Footprint" ""
+		(property "Footprint" "Capacitor_THT:C_Radial_D4.0mm_H7.0mm_P1.50mm"
 			(at 89.8652 102.87 0)
 			(effects
@@
 		(dnp no)
 		(fields_autoplaced yes)
-		(property "Reference" "SENS"
+		(property "Reference" "SENS1"
 			(at 166.37 129.5399 0)
 			(effects
@@
 			)
 		)
-		(property "Footprint" "Resistor_SMD:R_0201_0603Metric_Pad0.64x0.40mm_HandSolder"
+		(property "Footprint" "Resistor_SMD:R_2816_7142Metric_Pad3.20x4.45mm_HandSolder"
 			(at 162.052 130.81 90)
 			(effects
@@
 			(project "bhm"
 				(path "/6523cac7-11e3-4c79-8b92-51f4f81b827e"
-					(reference "SENS")
+					(reference "SENS1")
 					(unit 1)
 				)
@@
 		(dnp no)
 		(fields_autoplaced yes)
-		(property "Reference" "PosBatt"
+		(property "Reference" "PosBatt1"
 			(at 187.96 63.4999 0)
 			(effects
@@
 			)
 		)
-		(property "Footprint" ""
+		(property "Footprint" "1_Custom_Pads:bhm_large_power_pad"
 			(at 185.42 64.77 0)
 			(effects
@@
 			(project "bhm"
 				(path "/6523cac7-11e3-4c79-8b92-51f4f81b827e"
-					(reference "PosBatt")
+					(reference "PosBatt1")
 					(unit 1)
 				)
@@
 	(symbol
 		(lib_id "Connector_Generic:Conn_01x04")
-		(at 133.35 127 270)
+		(at 133.35 132.08 270)
 		(unit 1)
 		(exclude_from_sim no)
@@
 		(fields_autoplaced yes)
 		(property "Reference" "J1"
-			(at 132.08 130.81 90)
-			(effects
-				(font
-					(size 1.27 1.27)
-				)
-			)
-		)
-		(property "Value" "Conn_01x04"
-			(at 132.08 133.35 90)
+			(at 132.08 135.89 90)
+			(effects
+				(font
+					(size 1.27 1.27)
+				)
+			)
+		)
+		(property "Value" "SSD1306"
+			(at 132.08 138.43 90)
 			(effects
 				(font
@@
 		)
 		(property "Footprint" "Connector_PinHeader_2.54mm:PinHeader_1x04_P2.54mm_Vertical"
-			(at 133.35 127 0)
+			(at 133.35 132.08 0)
 			(effects
 				(font
@@
 		)
 		(property "Datasheet" "~"
-			(at 133.35 127 0)
+			(at 133.35 132.08 0)
 			(effects
 				(font
@@
 		)
 		(property "Description" "Generic connector, single row, 01x04, script generated (kicad-library-utils/schlib/autogen/connector/)"
-			(at 133.35 127 0)
-			(effects
-				(font
+			(at 133.35 132.08 0)
+			(effects
+				(font
